File: KiCAD/7PB.kicad_sch (KiCad schematic)
At the start: 44 parts, among them J1 Connector, J2 Connector, Q1 BC547, Q2 BC547, Q3 BC547, Q4 BC547, Q5 BC547, Q6 BC547, Q7 BC547

Commit message: Update
Changed lines of the file:
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@@
   (junction (at 91.44 76.2) (diameter 0) (color 0 0 0 0)
   )
+  (junction (at 35.56 63.5) (diameter 0) (color 0 0 0 0)
+  )
   (junction (at 190.5 76.2) (diameter 0) (color 0 0 0 0)
   )
@@
   (junction (at 243.84 101.6) (diameter 0) (color 0 0 0 0)
   )
+  (junction (at 35.56 109.22) (diameter 0) (color 0 0 0 0)
+  )
   (junction (at 177.8 83.82) (diameter 0) (color 0 0 0 0)
   )
@@
     (stroke (width 0) (type default) (color 0 0 0 0))
   )
-  (wire (pts (xy 30.48 109.22) (xy 45.72 109.22))
+  (wire (pts (xy 30.48 109.22) (xy 35.56 109.22))
     (stroke (width 0) (type default) (color 0 0 0 0))
   )
@@
     (stroke (width 0) (type default) (color 0 0 0 0))
   )
+  (wire (pts (xy 35.56 109.22) (xy 45.72 109.22))
+    (stroke (width 0) (type default) (color 0 0 0 0))
+  )
   (wire (pts (xy 71.12 76.2) (xy 78.74 76.2))
     (stroke (width 0) (type default) (color 0 0 0 0))
@@
     (stroke (width 0) (type default) (color 0 0 0 0))
   )
-  (wire (pts (xy 30.48 63.5) (xy 58.42 63.5))
+  (wire (pts (xy 30.48 63.5) (xy 35.56 63.5))
     (stroke (width 0) (type default) (color 0 0 0 0))
   )
@@
   )
   (wire (pts (xy 134.62 101.6) (xy 144.78 101.6))
+    (stroke (width 0) (type default) (color 0 0 0 0))
+  )
+  (wire (pts (xy 35.56 63.5) (xy 58.42 63.5))
     (stroke (width 0) (type default) (color 0 0 0 0))
   )
@@
     (pin "2")
   )
+  (symbol (lib_id "power:PWR_FLAG") (at 35.56 109.22 180) (unit 1)
+    (in_bom yes) (on_board yes) (fields_autoplaced)
+    (property "Reference" "#FLG0101" (id 0) (at 35.56 111.125 0)
+      (effects (font (size 1.27 1.27)) hide)
+    )
+    (property "Value" "PWR_FLAG" (id 1) (at 35.56 114.3 0))
+    (property "Footprint" "" (id 2) (at 35.56 109.22 0)
+      (effects (font (size 1.27 1.27)) hide)
+    )
+    (property "Datasheet" "~" (id 3) (at 35.56 109.22 0)
+      (effects (font (size 1.27 1.27)) hide)
+    )
+    (pin "1")
+  )
   (symbol (lib_id "Device:LED") (at 190.5 97.79 90) (unit 1)
     (in_bom yes) (on_board yes) (fields_autoplaced)
@@
     (pin "3")
   )
+  (symbol (lib_id "power:PWR_FLAG") (at 35.56 63.5 0) (unit 1)
+    (in_bom yes) (on_board yes) (fields_autoplaced)
+    (property "Reference" "#FLG0102" (id 0) (at 35.56 61.595 0)
+      (effects (font (size 1.27 1.27)) hide)
+    )
+    (property "Value" "PWR_FLAG" (id 1) (at 35.56 58.42 0))
+    (property "Footprint" "" (id 2) (at 35.56 63.5 0)
+      (effects (font (size 1.27 1.27)) hide)
+    )
+    (property "Datasheet" "~" (id 3) (at 35.56 63.5 0)
+      (effects (font (size 1.27 1.27)) hide)
+    )
+    (pin "1")
+  )
   (symbol (lib_id "Device:R") (at 190.5 69.85 0) (unit 1)
     (in_bom yes) (on_board yes) (fields_autoplaced)
@@
   )
   (symbol_instances
+    (path "/a1cec917-e27d-4439-bb48-9e26337e2ec5"
+      (reference "#FLG0101") (unit 1) (value "PWR_FLAG") (footprint "")
+    )
+    (path "/e7e9af52-81ac-45b0-8d47-90f62efd5d0d"
+      (reference "#FLG0102") (unit 1) (value "PWR_FLAG") (footprint "")
+    )
     (path "/d1900729-d56b-4976-aa55-9cc260dc60e7"
       (reference "#PWR01") (unit 1) (value "+9V") (footprint "")
