File: KiCAD/7PB.kicad_pcb (KiCad board)
At the start: 2 copper layers, 124.7 x 18 mm, 44 parts, among them J1 Connector, J2 Connector, Q1 BC547, Q2 BC547, Q3 BC547, Q4 BC547, Q5 BC547, Q6 BC547, Q7 BC547

Commit message: Update
Routing:
- net Net-(C4-Pad1): track 13.8 -> 17.2 mm
- net Net-(D5-Pad2): track 3.89 -> 3.26 mm
Other:
- board text added: "7PB"

Commit message: Update
Routing:
- added copper zone on B.Cu, net +9V
- removed copper zone on F.Cu, net +9V
- removed copper zone on F.Cu, net GND
